Commit message: Refactor tank room environment and add parallel GPU trainer

File: assets/tank_car.xacro (robot description, xacro)
@@ -1,106 +1,211 @@
 <?xml version="1.0"?>
-<robot xmlns:xacro="http://www.ros.org/wiki/xacro" name="tank_car">
-  <material name="platform_gray">
-    <color rgba="0.42 0.44 0.48 1.0"/>
+<robot name="tank_car" xmlns:xacro="http://www.ros.org/wiki/xacro">
+  <!--
+    Updated XACRO model of a very small tracked tank-like car.
+    Changes from the first version:
+    - Overall footprint is now about 10 cm x 15 cm (width x length).
+    - Lower ride height / less tall stance.
+    - Decorative motors moved UNDER the platform instead of sticking outside.
+    Notes:
+    - The center platform/chassis stays narrower than the full vehicle, like in the reference image.
+    - Tracks are still simplified as rigid boxes for URDF/XACRO visualization/collision.
+  -->
+  <xacro:property name="pi" value="3.1415926535897931"/>
+  <!-- Main dimensions (meters) -->
+  <!-- Narrow center platform, with total vehicle footprint ~0.10 m wide x 0.15 m long -->
+  <xacro:property name="body_length" value="0.10"/>
+  <xacro:property name="body_width"  value="0.05"/>
+  <xacro:property name="body_height" value="0.008"/>
+  <xacro:property name="body_ground_clearance" value="0.030"/>
+  <!-- Track + wheel geometry -->
+  <xacro:property name="track_width"       value="0.025"/>
+  <xacro:property name="wheel_radius"      value="0.022"/>
+  <xacro:property name="wheel_thickness"   value="0.008"/>
+  <xacro:property name="wheelbase"         value="0.106"/>
+  <xacro:property name="track_loop_length" value="${wheelbase + 2.0*wheel_radius}"/>
+  <xacro:property name="track_loop_height" value="${2.0*wheel_radius}"/>
+  <xacro:property name="track_center_y"    value="${body_width/2.0 + track_width/2.0 + 0.05}"/>
+  <!-- Derived positions -->
+  <xacro:property name="body_center_z" value="${body_ground_clearance + body_height/2.0}"/>
+  <xacro:property name="wheel_center_rel_z" value="${wheel_radius - body_center_z}"/>
+  <xacro:property name="front_x" value="${ wheelbase/2.0}"/>
+  <xacro:property name="rear_x"  value="${-wheelbase/2.0}"/>
+  <!-- Decorative motors now tucked under the platform -->
+  <xacro:property name="motor_radius" value="0.010"/>
+  <xacro:property name="motor_length" value="0.018"/>
+  <xacro:property name="motor_inset_y" value="${body_width/2.0 - motor_length/2.0 - 0.002}"/>
+  <xacro:property name="motor_underbody_z" value="${-body_height/2.0 - motor_radius}"/>
+  <!-- Masses -->
+  <xacro:property name="body_mass"        value="0.40"/>
+  <xacro:property name="wheel_mass"       value="0.03"/>
+  <xacro:property name="track_mass"       value="0.05"/>
+  <xacro:property name="motor_mass"       value="0.04"/>
+  <!-- Materials -->
+  <material name="silver">
+    <color rgba="0.80 0.80 0.82 1.0"/>
   </material>
-  <material name="track_black">
-    <color rgba="0.08 0.08 0.08 1.0"/>
+  <material name="dark_gray">
+    <color rgba="0.20 0.20 0.22 1.0"/>
   </material>
-  <material name="motor_blue">
-    <color rgba="0.10 0.24 0.62 1.0"/>
+  <material name="black">
+    <color rgba="0.05 0.05 0.05 1.0"/>
   </material>
-  <material name="free_wheel_silver">
-    <color rgba="0.72 0.72 0.74 1.0"/>
-  </material>
-  <xacro:property name="body_len" value="0.10"/>
-  <xacro:property name="body_wid" value="0.05"/>
-  <xacro:property name="body_thk" value="0.02"/>
-  <xacro:property name="lift" value="0.05"/>
-  <xacro:property name="wheel_r" value="0.010"/>
-  <xacro:property name="wheel_t" value="0.008"/>
-  <xacro:property name="wheel_y" value="0.043"/>
-  <xacro:property name="wheel_x" value="0.020"/>
-  <xacro:property name="track_len" value="0.085"/>
-  <xacro:property name="track_wid" value="0.012"/>
-  <xacro:property name="track_thk" value="0.007"/>
-  <link name="base_link">
+  <xacro:macro name="box_inertial" params="mass x y z">
     <inertial>
-      <origin xyz="0 0 ${lift + body_thk/2}" rpy="0 0 0"/>
-      <mass value="1.6"/>
-      <inertia ixx="0.0034" ixy="0" ixz="0" iyy="0.0020" iyz="0" izz="0.0047"/>
+      <origin xyz="0 0 0" rpy="0 0 0"/>
+      <mass value="${mass}"/>
+      <inertia
+        ixx="${mass*(y*y + z*z)/12.0}"
+        ixy="0.0"
+        ixz="0.0"
+        iyy="${mass*(x*x + z*z)/12.0}"
+        iyz="0.0"
+        izz="${mass*(x*x + y*y)/12.0}"/>
     </inertial>
+  </xacro:macro>
+  <xacro:macro name="cylinder_inertial" params="mass radius length">
+    <inertial>
+      <!-- Cylinder axis is rotated onto the Y-axis to match the wheel axle direction -->
+      <origin xyz="0 0 0" rpy="${pi/2} 0 0"/>
+      <mass value="${mass}"/>
+      <inertia
+        ixx="${mass*(3.0*radius*radius + length*length)/12.0}"
+        ixy="0.0"
+        ixz="0.0"
+        iyy="${mass*(3.0*radius*radius + length*length)/12.0}"
+        iyz="0.0"
+        izz="${0.5*mass*radius*radius}"/>
+    </inertial>
+  </xacro:macro>
+  <xacro:macro name="wheel_link" params="name">
+    <link name="${name}">
+      <xacro:cylinder_inertial mass="${wheel_mass}" radius="${wheel_radius}" length="${wheel_thickness}"/>
+      <visual>
+        <origin xyz="0 0 0" rpy="${pi/2} 0 0"/>
+        <geometry>
+          <cylinder radius="${wheel_radius}" length="${wheel_thickness}"/>
+        </geometry>
+        <material name="silver"/>
+      </visual>
+      <collision>
+        <origin xyz="0 0 0" rpy="${pi/2} 0 0"/>
+        <geometry>
+          <cylinder radius="${wheel_radius}" length="${wheel_thickness}"/>
+        </geometry>
+      </collision>
+    </link>
+  </xacro:macro>
+  <xacro:macro name="track_link" params="name">
+    <link name="${name}">
+      <xacro:box_inertial mass="${track_mass}" x="${track_loop_length}" y="${track_width}" z="${track_loop_height}"/>
+      <visual>
+        <origin xyz="0 0 0" rpy="0 0 0"/>
+        <geometry>
+          <box size="${track_loop_length} ${track_width} ${track_loop_height}"/>
+        </geometry>
+        <material name="black"/>
+      </visual>
+      <collision>
+        <origin xyz="0 0 0" rpy="0 0 0"/>
+        <geometry>
+          <box size="${track_loop_length} ${track_width} ${track_loop_height}"/>
+        </geometry>
+      </collision>
+    </link>
+  </xacro:macro>
+  <xacro:macro name="motor_link" params="name">
+    <link name="${name}">
+      <xacro:cylinder_inertial mass="${motor_mass}" radius="${motor_radius}" length="${motor_length}"/>
+      <visual>
+        <origin xyz="0 0 0" rpy="${pi/2} 0 0"/>
+        <geometry>
+          <cylinder radius="${motor_radius}" length="${motor_length}"/>
+        </geometry>
+        <material name="dark_gray"/>
+      </visual>
+      <collision>
+        <origin xyz="0 0 0" rpy="${pi/2} 0 0"/>
+        <geometry>
+          <cylinder radius="${motor_radius}" length="${motor_length}"/>
+        </geometry>
+      </collision>
+    </link>
+  </xacro:macro>
+  <link name="base_footprint"/>
+  <link name="chassis">
+    <xacro:box_inertial mass="${body_mass}" x="${body_length}" y="${body_width}" z="${body_height}"/>
     <visual>
-      <origin xyz="0 0 ${lift + body_thk/2}" rpy="0 0 0"/>
+      <origin xyz="0 0 0" rpy="0 0 0"/>
       <geometry>
-        <box size="${body_wid} ${body_len} ${body_thk}"/>
+        <box size="${body_length} ${body_width} ${body_height}"/>
       </geometry>
-      <material name="platform_gray"/>
+      <material name="silver"/>
     </visual>
     <collision>
-      <origin xyz="0 0 ${lift + body_thk/2}" rpy="0 0 0"/>
+      <origin xyz="0 0 0" rpy="0 0 0"/>
       <geometry>
-        <box size="${body_wid} ${body_len} ${body_thk}"/>
-      </geometry>
-    </collision>
-    <visual>
-      <origin xyz="${-wheel_x} 0 ${track_thk/2}" rpy="0 0 0"/>
-      <geometry>
-        <box size="${track_wid} ${track_len} ${track_thk}"/>
-      </geometry>
-      <material name="track_black"/>
-    </visual>
-    <collision>
-      <origin xyz="${-wheel_x} 0 ${track_thk/2}" rpy="0 0 0"/>
-      <geometry>
-        <box size="${track_wid} ${track_len} ${track_thk}"/>
-      </geometry>
-    </collision>
-    <visual>
-      <origin xyz="${wheel_x} 0 ${track_thk/2}" rpy="0 0 0"/>
-      <geometry>
-        <box size="${track_wid} ${track_len} ${track_thk}"/>
-      </geometry>
-      <material name="track_black"/>
-    </visual>
-    <collision>
-      <origin xyz="${wheel_x} 0 ${track_thk/2}" rpy="0 0 0"/>
-      <geometry>
-        <box size="${track_wid} ${track_len} ${track_thk}"/>
+        <box size="${body_length} ${body_width} ${body_height}"/>
       </geometry>
     </collision>
   </link>
-  <xacro:macro name="wheel_link" params="name x y mat">
-    <link name="${name}">
-      <inertial>
-        <origin xyz="0 0 0" rpy="0 0 0"/>
-        <mass value="0.08"/>
-        <inertia ixx="0.000008" ixy="0" ixz="0" iyy="0.000004" iyz="0" izz="0.000008"/>
-      </inertial>
-      <visual>
-        <origin xyz="0 0 0" rpy="1.57079632679 0 0"/>
-        <geometry>
-          <cylinder radius="${wheel_r}" length="${wheel_t}"/>
-        </geometry>
-        <material name="${mat}"/>
-      </visual>
-      <collision>
-        <origin xyz="0 0 0" rpy="1.57079632679 0 0"/>
-        <geometry>
-          <cylinder radius="${wheel_r}" length="${wheel_t}"/>
-        </geometry>
-      </collision>
-    </link>
-    <joint name="${name}_joint" type="continuous">
-      <parent link="base_link"/>
-      <child link="${name}"/>
-      <origin xyz="${x} ${y} ${wheel_r}" rpy="0 0 0"/>
-      <axis xyz="0 1 0"/>
-    </joint>
-  </xacro:macro>
-  <!-- Motorized diagonal wheels: front-left and rear-right -->
-  <xacro:wheel_link name="wheel_front_left_motor" x="${-wheel_x}" y="${wheel_y}" mat="motor_blue"/>
-  <xacro:wheel_link name="wheel_rear_right_motor" x="${wheel_x}" y="${-wheel_y}" mat="motor_blue"/>
-  <!-- Free wheels: front-right and rear-left -->
-  <xacro:wheel_link name="wheel_front_right_free" x="${wheel_x}" y="${wheel_y}" mat="free_wheel_silver"/>
-  <xacro:wheel_link name="wheel_rear_left_free" x="${-wheel_x}" y="${-wheel_y}" mat="free_wheel_silver"/>
+  <joint name="base_footprint_to_chassis" type="fixed">
+    <parent link="base_footprint"/>
+    <child link="chassis"/>
+    <origin xyz="0 0 ${body_center_z}" rpy="0 0 0"/>
+  </joint>
+  <!-- Wheels / sprockets -->
+  <xacro:wheel_link name="front_left_drive_wheel"/>
+  <xacro:wheel_link name="rear_left_idler_wheel"/>
+  <xacro:wheel_link name="front_right_idler_wheel"/>
+  <xacro:wheel_link name="rear_right_drive_wheel"/>
+  <joint name="front_left_drive_joint" type="continuous">
+    <parent link="chassis"/>
+    <child link="front_left_drive_wheel"/>
+    <origin xyz="${front_x} ${ track_center_y} ${wheel_center_rel_z}" rpy="0 0 0"/>
+    <axis xyz="0 1 0"/>
+  </joint>
+  <joint name="rear_left_idler_joint" type="continuous">
+    <parent link="chassis"/>
+    <child link="rear_left_idler_wheel"/>
+    <origin xyz="${rear_x} ${ track_center_y} ${wheel_center_rel_z}" rpy="0 0 0"/>
+    <axis xyz="0 1 0"/>
+  </joint>
+  <joint name="front_right_idler_joint" type="continuous">
+    <parent link="chassis"/>
+    <child link="front_right_idler_wheel"/>
+    <origin xyz="${front_x} ${-track_center_y} ${wheel_center_rel_z}" rpy="0 0 0"/>
+    <axis xyz="0 1 0"/>
+  </joint>
+  <joint name="rear_right_drive_joint" type="continuous">
+    <parent link="chassis"/>
+    <child link="rear_right_drive_wheel"/>
+    <origin xyz="${rear_x} ${-track_center_y} ${wheel_center_rel_z}" rpy="0 0 0"/>
+    <axis xyz="0 1 0"/>
+  </joint>
+  <!-- Simplified rigid track bodies -->
+  <xacro:track_link name="left_track"/>
+  <xacro:track_link name="right_track"/>
+  <joint name="left_track_joint" type="fixed">
+    <parent link="chassis"/>
+    <child link="left_track"/>
+    <origin xyz="0 ${ track_center_y} ${wheel_center_rel_z}" rpy="0 0 0"/>
+  </joint>
+  <joint name="right_track_joint" type="fixed">
+    <parent link="chassis"/>
+    <child link="right_track"/>
+    <origin xyz="0 ${-track_center_y} ${wheel_center_rel_z}" rpy="0 0 0"/>
+  </joint>
+  <!-- Decorative motors tucked under the platform on the driven corners -->
+  <xacro:motor_link name="front_left_motor"/>
+  <xacro:motor_link name="rear_right_motor"/>
+  <joint name="front_left_motor_joint" type="fixed">
+    <parent link="chassis"/>
+    <child link="front_left_motor"/>
+    <origin xyz="${front_x} ${motor_inset_y} ${motor_underbody_z}" rpy="0 0 0"/>
+  </joint>
+  <joint name="rear_right_motor_joint" type="fixed">
+    <parent link="chassis"/>
+    <child link="rear_right_motor"/>
+    <origin xyz="${rear_x} ${-motor_inset_y} ${motor_underbody_z}" rpy="0 0 0"/>
+  </joint>
 </robot>
